Commit message: TODO：新模型Z轴足端力被小腿Z轴分担了，因为他们重合在一起

File: resources/robots/buptDog/urdf/robot.urdf (robot description, URDF)
Before this commit: robot bupt_dog, 18 links, 17 joints
Links:
- removed link base
- link FL_FOOT: mass 0.06 -> 0.0; geometry collision sphere radius=0.02144; visual sphere radius=0.02144
- link FL_KNEE: mass 0.157 -> 0.22; geometry collision box size=0.02977 0.0225 0.228; visual box size=0.02977 0.0225 0.228
- link FL_X: mass 1.508 -> 1.440087; geometry collision cylinder length=0.1031 radius=0.046; visual cylinder length=0.1031 radius=0.046
- link FL_Y: mass 0.272 -> 0.272466; geometry collision box size=0.044 0.033 0.215; visual box size=0.044 0.033 0.215
- link FR_FOOT: mass 0.06 -> 0.0; geometry collision sphere radius=0.02144; visual sphere radius=0.02144
- link FR_KNEE: mass 0.157 -> 0.22; geometry collision box size=0.02977 0.0225 0.228; visual box size=0.02977 0.0225 0.228
- link FR_X: mass 1.508 -> 1.440087; geometry collision cylinder length=0.1031 radius=0.046; visual cylinder length=0.1031 radius=0.046
- link FR_Y: mass 0.272 -> 0.272466; geometry collision box size=0.044 0.033 0.215; visual box size=0.044 0.033 0.215
- link HL_FOOT: mass 0.06 -> 0.0; geometry collision sphere radius=0.02144; visual sphere radius=0.02144
- link HL_KNEE: mass 0.157 -> 0.22; geometry collision box size=0.02977 0.0225 0.228; visual box size=0.02977 0.0225 0.228
- link HL_X: mass 1.508 -> 1.440087; geometry collision cylinder length=0.1031 radius=0.046; visual cylinder length=0.1031 radius=0.046
- link HL_Y: mass 0.272 -> 0.272466; geometry collision box size=0.044 0.033 0.215; visual box size=0.044 0.033 0.215
- link HR_FOOT: mass 0.06 -> 0.0; geometry collision sphere radius=0.02144; visual sphere radius=0.02144
- link HR_KNEE: mass 0.157 -> 0.22; geometry collision box size=0.02977 0.0225 0.228; visual box size=0.02977 0.0225 0.228
- link HR_X: mass 1.508 -> 1.440087; geometry collision cylinder length=0.1031 radius=0.046; visual cylinder length=0.1031 radius=0.046
- link HR_Y: mass 0.272 -> 0.272466; geometry collision box size=0.044 0.033 0.215; visual box size=0.044 0.033 0.215
Joints:
- removed joint floating_base
- joint FL_FOOT_joint: origin xyz=0.0 0.0 -0.22799999999999998 rpy=0.0 0.0 0.0 -> xyz=0.0 0.0 -0.228 rpy=0.0 0.0 0.0
- joint FL_KNEE_joint: limit lower=-2.6965336943312392 upper=-0.9162978572970231 effort=33.5 velocity=21 -> lower=-2.792526803190927 upper=-0.6108652381980153 effort=33.5 velocity=21
- joint FL_X_joint: limit lower=-0.8028514559173915 upper=0.8028514559173915 effort=33.5 velocity=21 -> lower=-0.6981317007977318 upper=0.6981317007977318 effort=33.5 velocity=21
- joint FL_Y_joint: limit lower=-1.0471975511965976 upper=4.1887902047863905 effort=33.5 velocity=21 -> lower=-0.17453292519943295 upper=2.0943951023931953 effort=33.5 velocity=21; origin xyz=0.0 0.0991 0.0 rpy=0.0 0.0 0.0 -> xyz=0.0 0.1216 0.0 rpy=0.0 0.0 0.0
- joint FR_FOOT_joint: origin xyz=0.0 0.0 -0.22799999999999998 rpy=0.0 0.0 0.0 -> xyz=0.0 0.0 -0.228 rpy=0.0 0.0 0.0
- joint FR_KNEE_joint: limit lower=-2.6965336943312392 upper=-0.9162978572970231 effort=33.5 velocity=21 -> lower=-2.792526803190927 upper=-0.6108652381980153 effort=33.5 velocity=21
- joint FR_X_joint: limit lower=-0.8028514559173915 upper=0.8028514559173915 effort=33.5 velocity=21 -> lower=-0.6981317007977318 upper=0.6981317007977318 effort=33.5 velocity=21
- joint FR_Y_joint: limit lower=-1.0471975511965976 upper=4.1887902047863905 effort=33.5 velocity=21 -> lower=-0.17453292519943295 upper=2.0943951023931953 effort=33.5 velocity=21; origin xyz=0.0 -0.0991 0.0 rpy=0.0 0.0 0.0 -> xyz=0.0 -0.1216 0.0 rpy=0.0 0.0 0.0
- joint HL_FOOT_joint: origin xyz=0.0 0.0 -0.22799999999999998 rpy=0.0 0.0 0.0 -> xyz=0.0 0.0 -0.228 rpy=0.0 0.0 0.0
- joint HL_KNEE_joint: limit lower=-2.6965336943312392 upper=-0.9162978572970231 effort=33.5 velocity=21 -> lower=-2.792526803190927 upper=-0.6108652381980153 effort=33.5 velocity=21
- joint HL_X_joint: limit lower=-0.8028514559173915 upper=0.8028514559173915 effort=33.5 velocity=21 -> lower=-0.6981317007977318 upper=0.6981317007977318 effort=33.5 velocity=21
- joint HL_Y_joint: limit lower=-1.0471975511965976 upper=4.1887902047863905 effort=33.5 velocity=21 -> lower=-0.17453292519943295 upper=2.0943951023931953 effort=33.5 velocity=21; origin xyz=0.0 0.0991 0.0 rpy=0.0 0.0 0.0 -> xyz=0.0 0.1216 0.0 rpy=0.0 0.0 0.0
- joint HR_FOOT_joint: origin xyz=0.0 0.0 -0.22799999999999998 rpy=0.0 0.0 0.0 -> xyz=0.0 0.0 -0.228 rpy=0.0 0.0 0.0
- joint HR_KNEE_joint: limit lower=-2.6965336943312392 upper=-0.9162978572970231 effort=33.5 velocity=21 -> lower=-2.792526803190927 upper=-0.6108652381980153 effort=33.5 velocity=21
- joint HR_X_joint: limit lower=-0.8028514559173915 upper=0.8028514559173915 effort=33.5 velocity=21 -> lower=-0.6981317007977318 upper=0.6981317007977318 effort=33.5 velocity=21
- joint HR_Y_joint: limit lower=-1.0471975511965976 upper=4.1887902047863905 effort=33.5 velocity=21 -> lower=-0.17453292519943295 upper=2.0943951023931953 effort=33.5 velocity=21; origin xyz=0.0 -0.0991 0.0 rpy=0.0 0.0 0.0 -> xyz=0.0 -0.1216 0.0 rpy=0.0 0.0 0.0

Commit message: 新模型修复：足端惯性矩阵设置 2+2训练跑通

File: resources/robots/buptDog/urdf/robot.urdf (robot description, URDF)
Before this commit: robot bupt_dog, 17 links, 16 joints
Links:
- link FL_FOOT: mass 0.0 -> 0.06
- link FR_FOOT: mass 0.0 -> 0.06
- link HL_FOOT: mass 0.0 -> 0.06
- link HR_FOOT: mass 0.0 -> 0.06
